File: Circuit Designs/golgi_tendon_organ.kicad_sch (KiCad schematic)
At the start: 9 parts

Commit message: deleted previous version files
Parts:
- C154, C155, C156, C157: renamed from C?; footprint Capacitor_SMD:C_0402_1005Metric -> CoF_Capacitor:C-0402
- R87, R88, R89, R90: renamed from R?; footprint Resistor_SMD:R_0402_1005Metric -> CoF_Resistor:R-0402
- gave numbers to parts that had none: 1
Changed lines of the file:
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@@
   (junction (at 132.08 104.14) (diameter 0) (color 0 0 0 0)
   )
+  (junction (at 106.68 104.14) (diameter 0) (color 0 0 0 0)
+  )
   (junction (at 168.91 71.12) (diameter 0) (color 0 0 0 0)
   )
@@
     (stroke (width 0) (type default) (color 0 0 0 0))
   )
-  (wire (pts (xy 102.87 104.14) (xy 124.46 104.14))
+  (wire (pts (xy 102.87 104.14) (xy 106.68 104.14))
     (stroke (width 0) (type default) (color 0 0 0 0))
   )
@@
     (stroke (width 0) (type default) (color 0 0 0 0))
   )
+  (wire (pts (xy 106.68 104.14) (xy 106.68 105.41))
+    (stroke (width 0) (type default) (color 0 0 0 0))
+  )
   (wire (pts (xy 184.15 71.12) (xy 184.15 85.09))
     (stroke (width 0) (type default) (color 0 0 0 0))
@@
     (stroke (width 0) (type default) (color 0 0 0 0))
   )
+  (wire (pts (xy 106.68 104.14) (xy 124.46 104.14))
+    (stroke (width 0) (type default) (color 0 0 0 0))
+  )
   (image (at 38.1 30.48)
     (data
@@
   (symbol (lib_id "CoE_IntegratedCircuit:AS5047P") (at 146.05 88.9 0) (unit 1)
     (in_bom yes) (on_board yes)
-    (property "Reference" "U?" (id 0) (at 148.59 102.87 0)
+    (property "Reference" "U11" (id 0) (at 148.59 102.87 0)
       (effects (font (size 1.27 1.27)) (justify left))
     )
@@
   (symbol (lib_id "CoE_Resistor:10K") (at 124.46 76.2 0) (unit 1)
     (in_bom yes) (on_board yes)
-    (property "Reference" "R?" (id 0) (at 125.73 74.93 0)
+    (property "Reference" "R89" (id 0) (at 125.73 74.93 0)
       (effects (font (size 1.27 1.27)) (justify left))
     )
@@
       (effects (font (size 0.9906 0.9906)) (justify left))
     )
-    (property "Footprint" "Resistor_SMD:R_0402_1005Metric" (id 2) (at 124.46 66.04 0)
+    (property "Footprint" "CoF_Resistor:R-0402" (id 2) (at 124.46 66.04 0)
       (effects (font (size 1.27 1.27)) (justify bottom) hide)
     )
-    (property "Datasheet" "~" (id 3) (at 115.57 80.01 0)
+    (property "Datasheet" "~" (id 3) (at 124.46 92.71 0)
       (effects (font (size 1.27 1.27)) hide)
     )
@@
     (pin "2")
   )
-  (symbol (lib_name "10K_2") (lib_id "CoE_Resistor:10K") (at 115.57 76.2 0) (unit 1)
+  (symbol (lib_id "CoE_Resistor:10K") (at 115.57 76.2 0) (unit 1)
     (in_bom yes) (on_board yes)
-    (property "Reference" "R?" (id 0) (at 116.84 74.93 0)
+    (property "Reference" "R88" (id 0) (at 116.84 74.93 0)
       (effects (font (size 1.27 1.27)) (justify left))
     )
@@
       (effects (font (size 0.9906 0.9906)) (justify left))
     )
-    (property "Footprint" "Resistor_SMD:R_0402_1005Metric" (id 2) (at 115.57 66.04 0)
+    (property "Footprint" "CoF_Resistor:R-0402" (id 2) (at 115.57 66.04 0)
       (effects (font (size 1.27 1.27)) (justify bottom) hide)
     )
-    (property "Datasheet" "~" (id 3) (at 106.68 80.01 0)
+    (property "Datasheet" "~" (id 3) (at 115.57 92.71 0)
       (effects (font (size 1.27 1.27)) hide)
     )
@@
     (pin "2")
   )
-  (symbol (lib_name "10K_1") (lib_id "CoE_Resistor:10K") (at 106.68 76.2 0) (unit 1)
+  (symbol (lib_id "CoE_Resistor:10K") (at 106.68 76.2 0) (unit 1)
     (in_bom yes) (on_board yes)
-    (property "Reference" "R?" (id 0) (at 107.95 74.93 0)
+    (property "Reference" "R87" (id 0) (at 107.95 74.93 0)
       (effects (font (size 1.27 1.27)) (justify left))
     )
@@
       (effects (font (size 0.9906 0.9906)) (justify left))
     )
-    (property "Footprint" "Resistor_SMD:R_0402_1005Metric" (id 2) (at 106.68 66.04 0)
+    (property "Footprint" "CoF_Resistor:R-0402" (id 2) (at 106.68 66.04 0)
       (effects (font (size 1.27 1.27)) (justify bottom) hide)
     )
-    (property "Datasheet" "~" (id 3) (at 97.79 80.01 0)
+    (property "Datasheet" "~" (id 3) (at 106.68 92.71 0)
       (effects (font (size 1.27 1.27)) hide)
     )
@@
     (pin "2")
   )
-  (symbol (lib_name "10K_3") (lib_id "CoE_Resistor:10K") (at 124.46 93.98 0) (unit 1)
+  (symbol (lib_id "CoE_Resistor:10K") (at 124.46 93.98 0) (unit 1)
     (in_bom yes) (on_board yes)
-    (property "Reference" "R?" (id 0) (at 125.73 92.71 0)
+    (property "Reference" "R90" (id 0) (at 125.73 92.71 0)
       (effects (font (size 1.27 1.27)) (justify left))
     )
@@
       (effects (font (size 0.9906 0.9906)) (justify left))
     )
-    (property "Footprint" "Resistor_SMD:R_0402_1005Metric" (id 2) (at 124.46 83.82 0)
+    (property "Footprint" "CoF_Resistor:R-0402" (id 2) (at 124.46 83.82 0)
       (effects (font (size 1.27 1.27)) (justify bottom) hide)
     )
-    (property "Datasheet" "~" (id 3) (at 115.57 97.79 0)
+    (property "Datasheet" "~" (id 3) (at 124.46 110.49 0)
       (effects (font (size 1.27 1.27)) hide)
     )
@@
   (symbol (lib_id "CoE_Capacitor:1uF") (at 168.91 88.9 0) (unit 1)
     (in_bom yes) (on_board yes)
-    (property "Reference" "C?" (id 0) (at 169.545 86.36 0)
+    (property "Reference" "C154" (id 0) (at 169.545 86.36 0)
       (effects (font (size 1.27 1.27)) (justify left))
     )
@@
       (effects (font (size 0.9906 0.9906)) (justify left))
     )
-    (property "Footprint" "Capacitor_SMD:C_0402_1005Metric" (id 2) (at 168.91 78.74 0)
+    (property "Footprint" "CoF_Capacitor:C-0402" (id 2) (at 168.91 78.74 0)
       (effects (font (size 1.27 1.27)) (justify bottom) hide)
     )
-    (property "Datasheet" "~" (id 3) (at 168.91 88.9 0)
+    (property "Datasheet" "~" (id 3) (at 168.91 105.41 0)
       (effects (font (size 1.27 1.27)) hide)
     )
@@
   (symbol (lib_id "CoE_Capacitor:100nF") (at 184.15 88.9 0) (unit 1)
     (in_bom yes) (on_board yes)
-    (property "Reference" "C?" (id 0) (at 184.785 86.36 0)
+    (property "Reference" "C156" (id 0) (at 184.785 86.36 0)
       (effects (font (size 1.27 1.27)) (justify left))
     )
@@
       (effects (font (size 0.9906 0.9906)) (justify left))
     )
-    (property "Footprint" "Capacitor_SMD:C_0402_1005Metric" (id 2) (at 184.15 78.74 0)
+    (property "Footprint" "CoF_Capacitor:C-0402" (id 2) (at 184.15 78.74 0)
       (effects (font (size 1.27 1.27)) (justify bottom) hide)
     )
-    (property "Datasheet" "~" (id 3) (at 184.15 88.9 0)
+    (property "Datasheet" "~" (id 3) (at 184.15 105.41 0)
       (effects (font (size 1.27 1.27)) hide)
     )
@@
   (symbol (lib_id "CoE_Capacitor:1uF") (at 176.53 88.9 0) (unit 1)
     (in_bom yes) (on_board yes)
-    (property "Reference" "C?" (id 0) (at 177.165 86.36 0)
+    (property "Reference" "C155" (id 0) (at 177.165 86.36 0)
       (effects (font (size 1.27 1.27)) (justify left))
     )
@@
       (effects (font (size 0.9906 0.9906)) (justify left))
     )
-    (property "Footprint" "Capacitor_SMD:C_0402_1005Metric" (id 2) (at 176.53 78.74 0)
+    (property "Footprint" "CoF_Capacitor:C-0402" (id 2) (at 176.53 78.74 0)
       (effects (font (size 1.27 1.27)) (justify bottom) hide)
     )
-    (property "Datasheet" "~" (id 3) (at 176.53 88.9 0)
+    (property "Datasheet" "~" (id 3) (at 176.53 105.41 0)
       (effects (font (size 1.27 1.27)) hide)
     )
@@
   (symbol (lib_id "CoE_Capacitor:100nF") (at 191.77 88.9 0) (unit 1)
     (in_bom yes) (on_board yes)
-    (property "Reference" "C?" (id 0) (at 192.405 86.36 0)
+    (property "Reference" "C157" (id 0) (at 192.405 86.36 0)
       (effects (font (size 1.27 1.27)) (justify left))
     )
@@
       (effects (font (size 0.9906 0.9906)) (justify left))
     )
-    (property "Footprint" "Capacitor_SMD:C_0402_1005Metric" (id 2) (at 191.77 78.74 0)
+    (property "Footprint" "CoF_Capacitor:C-0402" (id 2) (at 191.77 78.74 0)
       (effects (font (size 1.27 1.27)) (justify bottom) hide)
     )
-    (property "Datasheet" "~" (id 3) (at 191.77 88.9 0)
+    (property "Datasheet" "~" (id 3) (at 191.77 105.41 0)
       (effects (font (size 1.27 1.27)) hide)
     )
@@
     (pin "2")
   )
+  (symbol (lib_id "power:PWR_FLAG") (at 106.68 105.41 180) (unit 1)
+    (in_bom yes) (on_board yes)
+    (property "Reference" "#FLG0102" (id 0) (at 106.68 107.315 0)
+      (effects (font (size 1.27 1.27)) hide)
+    )
+    (property "Value" "PWR_FLAG" (id 1) (at 106.68 109.22 0))
+    (property "Footprint" "" (id 2) (at 106.68 105.41 0)
+      (effects (font (size 1.27 1.27)) hide)
+    )
+    (property "Datasheet" "~" (id 3) (at 106.68 105.41 0)
+      (effects (font (size 1.27 1.27)) hide)
+    )
+    (pin "1")
+  )
 )
