File: Circuit Designs/pectoralis_major.kicad_sch (KiCad schematic)
At the start: 33 parts

Commit message: deleted previous version files
Parts:
- C1, C10, C11, C12, C13, C14, C15, C16, C17, C18, C19, C2, C20, C3, C4, C5, C6, C7, C8, C9: renamed from C?; footprint Capacitor_SMD:C_0805_2012Metric -> CoF_Capacitor:C-0805
- C21, C22, C23, C24, C25, C26: renamed from C?; footprint Capacitor_SMD:C_0402_1005Metric -> CoF_Capacitor:C-0402
- gave numbers to parts that had none: 7
Connections:
- net powerDrivers/BATT- is gone; now on net GND: C1.2, C10.2, C11.2, C12.2, C13.2, C14.2, C15.2, C16.2, C17.2, C18.2, C19.2, C2.2, C20.2, C3.2, C4.2, C5.2, C6.2, C7.2, C8.2, C9.2, J1.10 (Pin_10), J1.12 (Pin_12), J1.14 (Pin_14), J1.16 (Pin_16), J1.2 (Pin_2), J1.4 (Pin_4), J1.6 (Pin_6), J1.8 (Pin_8)
Other:
- sheet powerDrivers ports: added none; removed BATT-
