File: Circuit Designs/pectoralis_major.kicad_sch (KiCad schematic)
At the start: 33 parts, among them J1 0524651671, J2 0533071071, J3 0533071071, J4 0524651071

Commit message: done all the packages and migrations. Now, time to start to route the module
Parts:
- J1: footprint (none) -> CoF_Connector:524651671
- J2, J3: footprint (none) -> CoF_Connector:0533071071
- J4: footprint (none) -> CoF_Connector:524651071
- SP1: renamed from TP1; footprint TestPoint:TestPoint_Keystone_5019_Minature -> CoF_Connector:SolderPt_2.5x4mm; now left out of the parts list
- SP2: renamed from TP2; footprint TestPoint:TestPoint_Keystone_5019_Minature -> CoF_Connector:SolderPt_2.5x4mm; now left out of the parts list
- SP3: renamed from TP3; footprint TestPoint:TestPoint_Keystone_5019_Minature -> CoF_Connector:SolderPt_2.5x4mm
